File: hardware/PCB/DigiSlatePlus-Power.kicad_sch (KiCad schematic)
At the start: 38 parts, among them J3 +8-24 Volt, J4 Battery, J5 Mains, Q3 FS8205A, U21 LM2596S-ADJ, U22 DW01A, U23 TP4056, U24 KA78M05_TO252, U25 LD1117S33TR_SOT223

Commit message: updated
Changed lines of the file:
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@@
+	)
+	(symbol
+		(lib_id "Graphic:Logo_Open_Hardware_Small")
+		(at 185.42 173.99 0)
+		(unit 1)
+		(exclude_from_sim yes)
+		(in_bom no)
+		(on_board no)
+		(dnp no)
+		(fields_autoplaced yes)
+		(property "Reference" "#SYM3"
+			(at 185.42 167.005 0)
+			(effects
+				(font
+					(size 1.27 1.27)
+				)
+				(hide yes)
+			)
+		)
+		(property "Value" "Logo_Open_Hardware_Small"
+			(at 185.42 179.705 0)
+			(effects
+				(font
+					(size 1.27 1.27)
+				)
+				(hide yes)
+			)
+		)
+		(property "Footprint" ""
+			(at 185.42 173.99 0)
+			(effects
+				(font
+					(size 1.27 1.27)
+				)
+				(hide yes)
+			)
+		)
+		(property "Datasheet" "~"
+			(at 185.42 173.99 0)
+			(effects
+				(font
+					(size 1.27 1.27)
+				)
+				(hide yes)
+			)
+		)
+		(property "Description" "Open Hardware logo, small"
+			(at 185.42 173.99 0)
+			(effects
+				(font
+					(size 1.27 1.27)
+				)
+				(hide yes)
+			)
+		)
+		(instances
+			(project "DigiSlatePlus"
+				(path "/dcb9cf24-5afa-4bbe-8afa-a00529143e4d/8d8c6cc3-ae5a-4a9a-87ce-71fd40365acc"
+					(reference "#SYM3")
+					(unit 1)
+				)
+			)
+		)
 	)
 	(symbol
