File: hardware/PCB/DigiSlatePlus.kicad_pcb (KiCad board)
At the start: 2 copper layers, 270 x 135.9 mm, 121 parts, among them J1 Serial, J10 IO7, J2 USB_B, J3 +8-24 Volt, J4 Battery, J5 Mains, J6 Mains, J7 Timecode IN, J8 Timecode OUT, J9 MISO, Q1 2N2222, Q2 2N2222, Q3 FS8205A, Q4 2N2222, SW1 RotaryEncoder-SW, SW2 1, SW3 1, SW4 1, SW5 1, SW6 BOOT, U1 ESP32-S3-WROOM-1, U10 SA15-11SRWA, U11 SA15-11SRWA, U12 SA15-11SRWA, U13 SA15-11SRWA, U14 SA15-11SRWA, U15 SA15-11SRWA, U16 MAX7219, U17 SA15-11SRWA, U18 SA15-11SRWA, U19 SA15-11SRWA, U2 DS3231M, U20 SA15-11SRWA, U21 LM2596S-ADJ, U22 DW01A, U23 TP4056, U24 KA78M05_TO252, U25 LD1117S33TR_SOT223, U3 SA15-11SRWA, U4 SA15-11SRWA, U5 SA15-11SRWA, U6 SA15-11SRWA, U7 MAX7219, U8 SA15-11SRWA, U9 SA15-11SRWA

Commit message: updated
Parts:
- added G***: LOGO, Logos:Open-Source-Hardware-Logo, B.Cu at (105.2, 96.0)
- J3: moved to B.Cu
- moved J3 1.31 mm to (331.4, 189.5), turned to -90 degrees
- moved RV3 0.92 mm to (241.0, 80.8)
Routing:
- net GND: track 0.00 -> 22.4 mm, vias 0 -> 10
- net SC-C: track 235.1 -> 244.9 mm
- net SC-D: track 231.9 -> 241.5 mm
- net C: track 269.5 -> 278.1 mm
- net SC-E: track 235.9 -> 244.4 mm, vias 3 -> 1
- net SW1: track 259.8 -> 267.6 mm
- net E: track 273.8 -> 281.3 mm
- net D: track 267.7 -> 275.1 mm
- net SW3: track 278.9 -> 286.0 mm
- net SW2: track 296.8 -> 303.9 mm
- net SW4: track 268.0 -> 274.3 mm
- net F1: track 84.5 -> 80.3 mm
- net +3.3V: track 487.1 -> 490.2 mm
- net SC-1: track 139.1 -> 142.0 mm
- net M2: track 77.8 -> 79.9 mm
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Other:
- board text added: "+3.3V"
- board text added: "+5V"
- board text added: "+7-24V"
- board text added: "BATTERY"
- board text added: "CLAP-SWITCH"
- board text added: "DigiSlate+"
- board text added: "LCD contrast"
- board text added: "Li-Ion 3.7V"
- board text added: "MAIN"
- board text added: "SERIAL"
- board text added: "Scene - Take"
- board text added: "Scene/Take LED brightness"
- board text added: "TC-IN"
- board text added: "TC-OUT"
- board text added: "Timecode"
- board text added: "Timecode LED brightness"
- board text added: "USB"
- board text added: "charge status"
- board text added: "https://DigiSlatePlus.github.io"
