File: hardware/PCB/DigiSlatePlus.kicad_sch (KiCad schematic)
At the start: 40 parts, among them J1 Serial, J10 IO7, J2 USB_B, J6 Mains, J7 Timecode IN, J8 Timecode OUT, J9 MISO, Q4 2N2222, SW1 RotaryEncoder-SW, SW2 1, SW3 1, SW4 1, SW5 1, SW6 BOOT, U1 ESP32-S3-WROOM-1, U2 DS3231M

Commit message: updated
Changed lines of the file:
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@@
+	)
+	(symbol
+		(lib_id "Graphic:Logo_Open_Hardware_Small")
+		(at 185.42 173.99 0)
+		(unit 1)
+		(exclude_from_sim no)
+		(in_bom no)
+		(on_board no)
+		(dnp no)
+		(fields_autoplaced yes)
+		(property "Reference" "#SYM1"
+			(at 185.42 167.005 0)
+			(effects
+				(font
+					(size 1.27 1.27)
+				)
+				(hide yes)
+			)
+		)
+		(property "Value" "Logo_Open_Hardware_Small"
+			(at 185.42 179.705 0)
+			(effects
+				(font
+					(size 1.27 1.27)
+				)
+				(hide yes)
+			)
+		)
+		(property "Footprint" ""
+			(at 185.42 173.99 0)
+			(effects
+				(font
+					(size 1.27 1.27)
+				)
+				(hide yes)
+			)
+		)
+		(property "Datasheet" "~"
+			(at 185.42 173.99 0)
+			(effects
+				(font
+					(size 1.27 1.27)
+				)
+				(hide yes)
+			)
+		)
+		(property "Description" "Open Hardware logo, small"
+			(at 185.42 173.99 0)
+			(effects
+				(font
+					(size 1.27 1.27)
+				)
+				(hide yes)
+			)
+		)
+		(property "Sim.Enable" "0"
+			(at 185.42 173.99 0)
+			(effects
+				(font
+					(size 1.27 1.27)
+				)
+				(hide yes)
+			)
+		)
+		(instances
+			(project ""
+				(path "/dcb9cf24-5afa-4bbe-8afa-a00529143e4d"
+					(reference "#SYM1")
+					(unit 1)
+				)
+			)
+		)
 	)
 	(symbol
