File: hardware/PCB/tc_display.kicad_sch (KiCad schematic)
At the start: 43 parts, among them Q1 2N2222, Q2 2N2222, U10 SA15-11SRWA, U11 SA15-11SRWA, U12 SA15-11SRWA, U13 SA15-11SRWA, U14 SA15-11SRWA, U15 SA15-11SRWA, U16 MAX7219, U17 SA15-11SRWA, U18 SA15-11SRWA, U19 SA15-11SRWA, U20 SA15-11SRWA, U3 SA15-11SRWA, U4 SA15-11SRWA, U5 SA15-11SRWA, U6 SA15-11SRWA, U7 MAX7219, U8 SA15-11SRWA, U9 SA15-11SRWA

Commit message: updated
Changed lines of the file:
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@@
+	)
+	(symbol
+		(lib_id "Graphic:Logo_Open_Hardware_Small")
+		(at 185.42 173.99 0)
+		(unit 1)
+		(exclude_from_sim yes)
+		(in_bom no)
+		(on_board no)
+		(dnp no)
+		(fields_autoplaced yes)
+		(property "Reference" "#SYM2"
+			(at 185.42 167.005 0)
+			(effects
+				(font
+					(size 1.27 1.27)
+				)
+				(hide yes)
+			)
+		)
+		(property "Value" "Logo_Open_Hardware_Small"
+			(at 185.42 179.705 0)
+			(effects
+				(font
+					(size 1.27 1.27)
+				)
+				(hide yes)
+			)
+		)
+		(property "Footprint" ""
+			(at 185.42 173.99 0)
+			(effects
+				(font
+					(size 1.27 1.27)
+				)
+				(hide yes)
+			)
+		)
+		(property "Datasheet" "~"
+			(at 185.42 173.99 0)
+			(effects
+				(font
+					(size 1.27 1.27)
+				)
+				(hide yes)
+			)
+		)
+		(property "Description" "Open Hardware logo, small"
+			(at 185.42 173.99 0)
+			(effects
+				(font
+					(size 1.27 1.27)
+				)
+				(hide yes)
+			)
+		)
+		(instances
+			(project "DigiSlatePlus"
+				(path "/dcb9cf24-5afa-4bbe-8afa-a00529143e4d/8aad025e-4bc0-4907-b517-9a6d83f1b6c4"
+					(reference "#SYM2")
+					(unit 1)
+				)
+			)
+		)
 	)
 	(symbol
